File: pcb/k83-controller.kicad_pcb (KiCad board)
At the start: 2 copper layers, 69.3 x 22.4 mm, 37 parts, among them J1 USB_A

Commit message: switch X2 and Y0 pins to match board
Parts:
- REF**: value Y0 -> X2
- REF**: value X2 -> Y0

Commit message: update to kicad 6
Other:
- net class Default removed
